Commit message: Added camera on top and human model. Transmission not working

File: turtlebot3_description/urdf/turtlebot3_blind.gazebo.xacro (robot description, xacro)
@@ -177,3 +177,18 @@
     </sensor>
   </gazebo>
+  <gazebo>
+    <plugin name="gazebo_ros_control" filename="libgazebo_ros_control.so">
+     <robotNamespace>/camera_joint_model</robotNamespace>
+     <!--<robotSimType>gazebo_ros_control/DefaultRobotHWSim</robotSimType>-->
+    </plugin>
+  </gazebo>
+  <transmission name="base_to_camera_trans">
+    <type>transmission_interface/SimpleTransmission</type>
+    <actuator name="motor1">
+     <mechanicalReduction>1</mechanicalReduction>
+    </actuator>
+    <joint name="camera_joint">
+     <hardwareInterface>hardware_interface/EffortJointInterface</hardwareInterface>
+    </joint>
+   </transmission>
 </robot>

File: turtlebot3_description/urdf/turtlebot3_blind.urdf.xacro (robot description, xacro)
@@ -164,12 +164,28 @@
     </inertial>
   </link>
-  <joint name="camera_joint" type="fixed">
+  <!-- I have added a person link/joint to put a model of the human (just visually, no inertias) -->
+  <!--
+  <link name="person_link">
+    <visual>
+     <origin xyz="-0.15 0 0" rpy="0 0 1.57"/>
+     <geometry>
+      <mesh filename="package://turtlebot3_gazebo/models/person_standing/meshes/standing.dae" />
+     </geometry>
+    </visual>
+  </link>
+  <joint name="person_joint" type="fixed">
+    <origin xyz="0 0 0" rpy="0 0 0"/>
+    <parent link="base_footprint"/>
+    <child link="person_link"/>
+  </joint>-->
+  <joint name="camera_joint" type="continuous">
     <origin xyz="0.064 -0.065 0.094" rpy="0 0 0"/>
     <parent link="base_link"/>
     <child link="camera_link"/>
+    <axis xyz="0 1 0"/>
   </joint>
   <link name="camera_link">
     <visual>
-     <origin xyz="0 0 0" rpy="1.57 0 1.57"/>
+     <origin xyz="-0.07 0.01 1.675" rpy="1.57 0 1.57"/>
       <geometry>
        <mesh filename="package://turtlebot3_description/meshes/sensors/r200.dae" />
@@ -183,11 +199,11 @@
     </collision>
     <!-- This inertial field needs doesn't contain reliable data!! -->
-<!--   <inertial>
-      <mass value="0.564" />
+    <inertial>
+      <mass value="0.001" /> <!-- 0.564 -->
       <origin xyz="0 0 0" />
       <inertia ixx="0.003881243" ixy="0.0" ixz="0.0"
                iyy="0.000498940" iyz="0.0"
                izz="0.003879257" />
-    </inertial>-->
+    </inertial>
   </link>
   <joint name="camera_rgb_joint" type="fixed">

Commit message: Turtlebot3 now working completely with moving head/camera and other adjustments to integrate with RGBD_VIA and Navigation branch

File: turtlebot3_description/urdf/turtlebot3_blind.gazebo.xacro (robot description, xacro)
@@ -58,5 +58,5 @@
       <odometryFrame>odom</odometryFrame>
       <odometrySource>world</odometrySource>
-      <publishOdomTF>true</publishOdomTF>
+      <publishOdomTF>false</publishOdomTF>
       <robotBaseFrame>base_footprint</robotBaseFrame>
       <publishWheelTF>false</publishWheelTF>
@@ -134,4 +134,6 @@
     </sensor>
   </gazebo>
+<!--CAMERA REAL SENSE-->
+<!--
   <gazebo reference="camera_rgb_frame">
     <sensor type="depth" name="realsense_R200">
@@ -177,18 +179,58 @@
     </sensor>
   </gazebo>
+-->
+<!--CAMERA ASUS-->
+    <gazebo reference="camera_rgb_frame">
+      <sensor type="depth" name="camera">
+        <always_on>true</always_on>
+        <update_rate>20.0</update_rate>
+        <camera>
+          <horizontal_fov>${60.0*3.141592/180.0}</horizontal_fov>
+          <image>
+            <format>B8G8R8</format>
+            <width>640</width>
+            <height>480</height>
+          </image>
+          <clip>
+            <near>0.05</near>
+            <far>8.0</far>
+          </clip>
+        </camera>
+        <plugin name="kinect_camera_controller" filename="libgazebo_ros_openni_kinect.so">
+          <cameraName>camera</cameraName>
+          <alwaysOn>true</alwaysOn>
+          <updateRate>10</updateRate>
+          <imageTopicName>rgb/image_raw</imageTopicName>
+          <depthImageTopicName>depth_registered/image_raw</depthImageTopicName>
+          <pointCloudTopicName>depth_registered/points</pointCloudTopicName>
+          <cameraInfoTopicName>rgb/camera_info</cameraInfoTopicName>
+          <depthImageCameraInfoTopicName>depth_registered/camera_info</depthImageCameraInfoTopicName>
+          <frameName>camera_depth_optical_frame</frameName>
+          <baseline>0.1</baseline>
+          <distortion_k1>0.0</distortion_k1>
+          <distortion_k2>0.0</distortion_k2>
+          <distortion_k3>0.0</distortion_k3>
+          <distortion_t1>0.0</distortion_t1>
+          <distortion_t2>0.0</distortion_t2>
+          <pointCloudCutoff>0.4</pointCloudCutoff>
+        </plugin>
+      </sensor>
+    </gazebo>
   <gazebo>
     <plugin name="gazebo_ros_control" filename="libgazebo_ros_control.so">
      <robotNamespace>/camera_joint_model</robotNamespace>
-     <!--<robotSimType>gazebo_ros_control/DefaultRobotHWSim</robotSimType>-->
-    </plugin>
-  </gazebo>
-  <transmission name="base_to_camera_trans">
-    <type>transmission_interface/SimpleTransmission</type>
-    <actuator name="motor1">
-     <mechanicalReduction>1</mechanicalReduction>
-    </actuator>
-    <joint name="camera_joint">
-     <hardwareInterface>hardware_interface/EffortJointInterface</hardwareInterface>
-    </joint>
-   </transmission>
+    </plugin>
+  </gazebo>
+  <gazebo>
+    <plugin name="p3d_base_controller" filename="libgazebo_ros_p3d.so"> <!-- sauravag.com/2017/06/how-to-get-ground-truth-pose-data-in-ros-gazebo/-->
+      <alwaysOn>true</alwaysOn>
+      <updateRate>50.0</updateRate>
+      <bodyName>base_footprint</bodyName>
+      <topicName>ground_truth/state</topicName>
+      <gaussianNoise>0.01</gaussianNoise>
+      <frameName>world</frameName>
+      <xyzOffsets>0 0 0</xyzOffsets>
+      <rpyOffsets>0 0 0</rpyOffsets>
+    </plugin>
+  </gazebo>
 </robot>

File: turtlebot3_description/urdf/turtlebot3_blind.urdf.xacro (robot description, xacro)
@@ -2,5 +2,5 @@
 <robot name="turtlebot3_waffle" xmlns:xacro="http://ros.org/wiki/xacro">
   <xacro:include filename="$(find turtlebot3_description)/urdf/common_properties.xacro"/>
-  <xacro:include filename="$(find turtlebot3_description)/urdf/turtlebot3_waffle.gazebo.xacro"/>
+  <xacro:include filename="$(find turtlebot3_description)/urdf/turtlebot3_blind.gazebo.xacro"/>
   <xacro:property name="r200_cam_rgb_px" value="0.005"/>
   <xacro:property name="r200_cam_rgb_py" value="0.018"/>
@@ -164,22 +164,26 @@
     </inertial>
   </link>
-  <!-- I have added a person link/joint to put a model of the human (just visually, no inertias) -->
-  <!--
-  <link name="person_link">
-    <visual>
-     <origin xyz="-0.15 0 0" rpy="0 0 1.57"/>
-     <geometry>
-      <mesh filename="package://turtlebot3_gazebo/models/person_standing/meshes/standing.dae" />
-     </geometry>
-    </visual>
-  </link>
-  <joint name="person_joint" type="fixed">
+<joint name="head_joint" type="fixed">
+  <!--<origin xyz="0.064 -0.065 0.094" rpy="0 0 0"/>-->
+  <!--<origin xyz="-0.07 0.075 1.674" rpy="0 0 0"/>-->
+  <origin xyz="0.00 0.012 1.76" rpy="0 0 0"/>
+  <parent link="base_link"/>
+  <child link="head_link"/>
+</joint>
+<link name="head_link">
+  <origin xyz="0 0 0" rpy="0 0 0"/>
+  <!-- This inertial field needs doesn't contain reliable data!! -->
+  <inertial>
+    <mass value="0.001" /> <!-- 0.564 -->
+    <origin xyz="0 0 0" />
+    <inertia ixx="0.0" ixy="0.0" ixz="0.0"
+             iyy="0.0" iyz="0.0"
+             izz="0.0" />
+  </inertial>
+</link>
+  <joint name="camera_joint" type="continuous">
+    <!--<origin xyz="0.064 -0.065 0.094" rpy="0 0 0"/>-->
     <origin xyz="0 0 0" rpy="0 0 0"/>
-    <parent link="base_footprint"/>
-    <child link="person_link"/>
-  </joint>-->
-  <joint name="camera_joint" type="continuous">
-    <origin xyz="0.064 -0.065 0.094" rpy="0 0 0"/>
-    <parent link="base_link"/>
+    <parent link="head_link"/>
     <child link="camera_link"/>
     <axis xyz="0 1 0"/>
@@ -187,8 +191,14 @@
   <link name="camera_link">
     <visual>
-     <origin xyz="-0.07 0.01 1.675" rpy="1.57 0 1.57"/>
+    <!--CAMERA ASUS-->
+    <origin xyz="0 0 0" rpy="0 0 0"/>
+    <geometry>
+     <mesh filename="package://turtlebot3_gazebo/models/asus_xtion_pro_camera/meshes/asus_xtion_pro_camera.dae" />
+    </geometry>
+    <!--CAMERA REAL SENSE-->
+     <!--<origin xyz="-0.07 0.01 1.675" rpy="1.57 0 1.57"/>
       <geometry>
        <mesh filename="package://turtlebot3_description/meshes/sensors/r200.dae" />
-      </geometry>
+      </geometry>-->
     </visual>
     <collision>
@@ -231,3 +241,26 @@
   </joint>
   <link name="camera_depth_optical_frame"/>
+  <!-- I have added a person link/joint to put a model of the human (just visually, no inertias) -->
+  <link name="person_link">
+    <visual>
+     <origin xyz="-0.15 0 0" rpy="0 0 1.57"/>
+     <geometry>
+      <mesh filename="package://turtlebot3_gazebo/models/person_standing/meshes/standing.dae" />
+     </geometry>
+    </visual>
+  </link>
+  <joint name="person_joint" type="fixed">
+    <origin xyz="0 0 0" rpy="0 0 0"/>
+    <parent link="base_footprint"/>
+    <child link="person_link"/>
+  </joint>
+  <transmission name="base_to_camera_trans">
+    <type>transmission_interface/SimpleTransmission</type>
+    <actuator name="motor1">
+     <mechanicalReduction>1</mechanicalReduction>
+    </actuator>
+    <joint name="camera_joint">
+     <hardwareInterface>hardware_interface/EffortJointInterface</hardwareInterface>
+    </joint>
+   </transmission>
 </robot>
